File: eagle/meduza01/meduza01.brd (EAGLE design)
At the start: 68.6 x 25.4 mm, 45 parts, among them U1 L3G4200D, U2 MMA8452QL, U3 MAG3110L, U4 MCP73831, U5 SD, U6 IRDA, Y1 8MHZ

Commit message: meduza01 board files
Parts:
- C1, C10, C101, C102, C103, C104, C105, C106, C107, C108, C7, C8, C9: device SparkFun:0603-CAP -> naut:0603
- C4: device SparkFun-Passives:0805 -> naut:0603
- R1, R10, R2, R8, R9: device SparkFun:0603-RES -> naut:0603
- R11, R3, R4, R5, R6, R7: device SparkFun-Resistors:0603-RES -> naut:0603
- U$6: device 0drom:QFP80P1200X1200X120-44N -> naut:QFP80P1200X1200X120-44N
- U2: device 0drom:QFN-16_0.5MM-EXTRA -> naut:QFN-16_0.5MM-EXTRA
- U3: device 0drom:DFN-10-EXTRA -> naut:DFN-10-EXTRA
- moved U$1 0.57 mm to (47.2, 12.0)
Routing:
- net GND: track 36.4 -> 23.4 mm
- net 3.3V: track 212.0 -> 213.5 mm
- net V_BATT: track 51.5 -> 50.8 mm
