File: eagle/meduza01/meduza01.sch (EAGLE design)
At the start: 45 parts, among them U1 L3G4200D, U2 MMA8452QL, U3 MAG3110L, U4 MCP73831, U5 SD, U6 IRDA, Y1 8MHZ

Commit message: meduza01 board files
Parts:
- C1, C10, C101, C102, C103, C104, C105, C106, C107, C108, C7, C8, C9: device SparkFun:CAP0603-CAP -> naut:CAP0603
- C4: device SparkFun-Passives:CAP0805 -> naut:CAP0603
- R1, R10, R2, R8, R9: device SparkFun:RESISTOR0603-RES -> naut:RESISTOR0603
- R11, R3, R4, R5, R6, R7: device SparkFun-Resistors:RESISTOR0603-RES -> naut:RESISTOR0603
- U$3: device 0drom:MCP1700T-3302E/TTSOT89MCP1700-3N -> naut:MCP1700T-3302E/TTSOT89MCP1700-3N
- U$6: device 0drom:PIC24FJ64GA004 -> naut:PIC24FJ64GA004
- U2: device 0drom:MMA8452QL -> naut:MMA8452QL
- U3: device 0drom:MAG3110L -> naut:MAG3110L
- U5: device 0drom:USD-SOCKETMOLEX47309 -> naut:USD-SOCKETMOLEX47309
- U6: device 0drom:TFDU6300TFDU6300 -> naut:TFDU6300TFDU6300
Changed lines of the file:
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@@
 <part name="GND5" library="SparkFun" deviceset="GND" device=""/>
 <part name="GND6" library="SparkFun" deviceset="GND" device=""/>
-<part name="C101" library="SparkFun" deviceset="CAP" device="0603-CAP"/>
-<part name="C102" library="SparkFun" deviceset="CAP" device="0603-CAP"/>
-<part name="C103" library="SparkFun" deviceset="CAP" device="0603-CAP"/>
-<part name="C104" library="SparkFun" deviceset="CAP" device="0603-CAP"/>
-<part name="C1" library="SparkFun" deviceset="CAP" device="0603-CAP"/>
+<part name="C101" library="naut" deviceset="CAP" device="0603"/>
+<part name="C102" library="naut" deviceset="CAP" device="0603"/>
+<part name="C103" library="naut" deviceset="CAP" device="0603"/>
+<part name="C104" library="naut" deviceset="CAP" device="0603"/>
+<part name="C1" library="naut" deviceset="CAP" device="0603"/>
 <part name="GND7" library="SparkFun" deviceset="GND" device=""/>
 <part name="GND8" library="SparkFun" deviceset="GND" device=""/>
@@
 <part name="P+8" library="SparkFun" deviceset="3.3V" device=""/>
 <part name="P+9" library="SparkFun" deviceset="3.3V" device=""/>
-<part name="C105" library="SparkFun" deviceset="CAP" device="0603-CAP"/>
+<part name="C105" library="naut" deviceset="CAP" device="0603"/>
 <part name="P+10" library="SparkFun" deviceset="3.3V" device=""/>
 <part name="GND12" library="SparkFun" deviceset="GND" device=""/>
-<part name="C7" library="SparkFun" deviceset="CAP" device="0603-CAP"/>
+<part name="C7" library="naut" deviceset="CAP" device="0603"/>
 <part name="GND13" library="SparkFun" deviceset="GND" device=""/>
-<part name="R1" library="SparkFun" deviceset="RESISTOR" device="0603-RES"/>
-<part name="R2" library="SparkFun" deviceset="RESISTOR" device="0603-RES"/>
+<part name="R1" library="naut" deviceset="RESISTOR" device="0603"/>
+<part name="R2" library="naut" deviceset="RESISTOR" device="0603"/>
 <part name="P+11" library="SparkFun" deviceset="3.3V" device=""/>
 <part name="GND14" library="SparkFun" deviceset="GND" device=""/>
 <part name="P+13" library="SparkFun" deviceset="3.3V" device=""/>
 <part name="GND15" library="SparkFun" deviceset="GND" device=""/>
-<part name="C8" library="SparkFun" deviceset="CAP" device="0603-CAP"/>
+<part name="C8" library="naut" deviceset="CAP" device="0603"/>
 <part name="GND16" library="SparkFun" deviceset="GND" device=""/>
-<part name="C9" library="SparkFun" deviceset="CAP" device="0603-CAP"/>
-<part name="C10" library="SparkFun" deviceset="CAP" device="0603-CAP"/>
+<part name="C9" library="naut" deviceset="CAP" device="0603"/>
+<part name="C10" library="naut" deviceset="CAP" device="0603"/>
 <part name="GND17" library="SparkFun" deviceset="GND" device=""/>
 <part name="GND18" library="SparkFun" deviceset="GND" device=""/>
-<part name="C106" library="SparkFun" deviceset="CAP" device="0603-CAP"/>
+<part name="C106" library="naut" deviceset="CAP" device="0603"/>
 <part name="GND19" library="SparkFun" deviceset="GND" device=""/>
 <part name="P+15" library="SparkFun" deviceset="3.3V" device=""/>
@@
 <part name="GND25" library="SparkFun" deviceset="GND" device=""/>
 <part name="GND26" library="SparkFun" deviceset="GND" device=""/>
-<part name="R3" library="SparkFun-Resistors" deviceset="RESISTOR" device="0603-RES"/>
-<part name="R4" library="SparkFun-Resistors" deviceset="RESISTOR" device="0603-RES"/>
+<part name="R3" library="naut" deviceset="RESISTOR" device="0603"/>
+<part name="R4" library="naut" deviceset="RESISTOR" device="0603"/>
 <part name="C2" library="SparkFun-Passives" deviceset="CAP" device="0805"/>
 <part name="GND27" library="SparkFun" deviceset="GND" device=""/>
@@
 <part name="JP2" library="SparkFun-Connectors" deviceset="M02" device="PTH"/>
 <part name="GND28" library="SparkFun" deviceset="GND" device=""/>
-<part name="R6" library="SparkFun-Resistors" deviceset="RESISTOR" device="0603-RES"/>
-<part name="R7" library="SparkFun-Resistors" deviceset="RESISTOR" device="0603-RES"/>
+<part name="R6" library="naut" deviceset="RESISTOR" device="0603"/>
+<part name="R7" library="naut" deviceset="RESISTOR" device="0603"/>
 <part name="GND30" library="SparkFun" deviceset="GND" device=""/>
-<part name="U5" library="0drom" deviceset="USD-SOCKET" device="MOLEX47309" value="SD"/>
+<part name="U5" library="naut" deviceset="USD-SOCKET" device="MOLEX47309" value="SD"/>
 <part name="GND31" library="SparkFun" deviceset="GND" device=""/>
 <part name="P+18" library="SparkFun" deviceset="3.3V" device=""/>
 <part name="U$5" library="SparkFun-Aesthetics" deviceset="5V" device=""/>
 <part name="GND24" library="SparkFun" deviceset="GND" device=""/>
-<part name="U6" library="0drom" deviceset="TFDU6300" device="TFDU6300" value="IRDA"/>
+<part name="U6" library="naut" deviceset="TFDU6300" device="TFDU6300" value="IRDA"/>
 <part name="GND37" library="SparkFun" deviceset="GND" device=""/>
 <part name="P+12" library="SparkFun" deviceset="3.3V" device=""/>
 <part name="Y1" library="SparkFun-FreqCtrl" deviceset="RESONATOR" device="8MHZ" value="8MHZ"/>
 <part name="GND38" library="SparkFun" deviceset="GND" device=""/>
-<part name="U3" library="0drom" deviceset="MAG3110" device="L"/>
-<part name="U2" library="0drom" deviceset="MMA8452Q" device="L"/>
-<part name="U$3" library="0drom" deviceset="MCP1700T-3302E/TT" device="SOT89MCP1700-3N" value="LDO"/>
-<part name="U$6" library="0drom" deviceset="PIC24FJ64GA004" device="" value="uC"/>
+<part name="U3" library="naut" deviceset="MAG3110" device="L"/>
+<part name="U2" library="naut" deviceset="MMA8452Q" device="L"/>
+<part name="U$3" library="naut" deviceset="MCP1700T-3302E/TT" device="SOT89MCP1700-3N" value="LDO"/>
+<part name="U$6" library="naut" deviceset="PIC24FJ64GA004" device="" value="uC"/>
 <part name="LED1" library="SparkFun-LED" deviceset="LED" device="1206"/>
 <part name="GND29" library="SparkFun" deviceset="GND" device=""/>
 <part name="P+14" library="SparkFun" deviceset="3.3V" device=""/>
-<part name="C107" library="SparkFun" deviceset="CAP" device="0603-CAP"/>
+<part name="C107" library="naut" deviceset="CAP" device="0603"/>
 <part name="GND32" library="SparkFun" deviceset="GND" device=""/>
 <part name="P+19" library="SparkFun" deviceset="3.3V" device=""/>
-<part name="C108" library="SparkFun" deviceset="CAP" device="0603-CAP"/>
+<part name="C108" library="naut" deviceset="CAP" device="0603"/>
 <part name="GND33" library="SparkFun" deviceset="GND" device=""/>
 <part name="P+20" library="SparkFun" deviceset="3.3V" device=""/>
 <part name="U$2" library="naut" deviceset="MCP9800" device=""/>
-<part name="C4" library="SparkFun-Passives" deviceset="CAP" device="0805"/>
+<part name="C4" library="naut" deviceset="CAP" device="0603"/>
 <part name="LED2" library="SparkFun-LED" deviceset="LED" device="1206"/>
-<part name="R5" library="SparkFun-Resistors" deviceset="RESISTOR" device="0603-RES"/>
+<part name="R5" library="naut" deviceset="RESISTOR" device="0603"/>
 <part name="GND34" library="SparkFun" deviceset="GND" device=""/>
 <part name="JP3" library="SparkFun-Connectors" deviceset="M14" device=""/>
 <part name="JP7" library="SparkFun-Connectors" deviceset="M14" device=""/>
-<part name="R8" library="SparkFun" deviceset="RESISTOR" device="0603-RES"/>
-<part name="R9" library="SparkFun" deviceset="RESISTOR" device="0603-RES"/>
-<part name="R10" library="SparkFun" deviceset="RESISTOR" device="0603-RES"/>
+<part name="R8" library="naut" deviceset="RESISTOR" device="0603"/>
+<part name="R9" library="naut" deviceset="RESISTOR" device="0603"/>
+<part name="R10" library="naut" deviceset="RESISTOR" device="0603"/>
 <part name="GND35" library="SparkFun" deviceset="GND" device=""/>
 <part name="LED3" library="SparkFun-LED" deviceset="LED" device="1206"/>
-<part name="R11" library="SparkFun-Resistors" deviceset="RESISTOR" device="0603-RES"/>
+<part name="R11" library="naut" deviceset="RESISTOR" device="0603"/>
 <part name="U$7" library="SparkFun-Aesthetics" deviceset="V_BATT" device=""/>
 <part name="U$1" library="naut" deviceset="MEDUZA01" device=""/>
